Commit message: disable mimic tag

File: src/curobo/content/assets/robot/soar_description/soar.urdf (robot description, URDF)
Before this commit: robot soar, 62 links, 61 joints
Joints:
- joint left_finger_joint: mimic joint=drive_joint multiplier=1 offset=0 -> (none)
- joint left_inner_knuckle_joint: mimic joint=drive_joint multiplier=1 offset=0 -> (none)
- joint right_finger_joint: mimic joint=drive_joint multiplier=1 offset=0 -> (none)
- joint right_inner_knuckle_joint: mimic joint=drive_joint multiplier=1 offset=0 -> (none)
- joint right_outer_knuckle_joint: mimic joint=drive_joint multiplier=1 offset=0 -> (none)

Commit message: apply moveit limit

File: src/curobo/content/assets/robot/soar_description/soar.urdf (robot description, URDF)
Before this commit: robot soar, 62 links, 61 joints
Joints:
- joint arm_joint1: limit lower=-6.283185307179586 upper=6.283185307179586 effort=42 velocity=3.14 -> lower=-2.6 upper=0.506 effort=42 velocity=2.826
- joint arm_joint2: limit lower=-2.059 upper=2.0944 effort=42 velocity=3.14 -> lower=-2.059 upper=2.0944 effort=42 velocity=2.826
- joint arm_joint3: limit lower=-6.283185307179586 upper=6.283185307179586 effort=19 velocity=3.14 -> lower=-3.141 upper=3.141 effort=19 velocity=2.86
- joint arm_joint4: limit lower=-0.19198 upper=3.927 effort=19 velocity=3.14 -> lower=-0.19198 upper=3.927 effort=19 velocity=2.826
- joint arm_joint5: limit lower=-6.283185307179586 upper=6.283185307179586 effort=19 velocity=3.14 -> lower=-3.141 upper=3.141 effort=19 velocity=2.826
- joint arm_joint6: limit lower=-1.69297 upper=3.141592653589793 effort=7 velocity=3.14 -> lower=-1.57 upper=3.141592653589793 effort=7 velocity=2.826
- joint arm_joint7: limit lower=-6.283185307179586 upper=6.283185307179586 effort=7 velocity=3.14 -> lower=-3.141 upper=3.141 effort=7 velocity=2.826
- joint torso_joint: limit lower=0.0 upper=0.41 effort=5000.0 velocity=10 -> lower=0.0 upper=0.41 effort=5000.0 velocity=0.1

Commit message: test

File: src/curobo/content/assets/robot/soar_description/soar.urdf (robot description, URDF)
Before this commit: robot soar, 62 links, 61 joints
Joints:
- joint drive_joint: type revolute -> fixed
- joint head_pan_joint: type revolute -> fixed
- joint head_tilt_joint: type revolute -> fixed
- joint left_finger_joint: type revolute -> fixed
- joint left_inner_knuckle_joint: type revolute -> fixed
- joint right_finger_joint: type revolute -> fixed
- joint right_inner_knuckle_joint: type revolute -> fixed
- joint right_outer_knuckle_joint: type revolute -> fixed
